File: kastle_arp_euro.kicad_sch (KiCad schematic)
At the start: 74 parts, among them J1 Conn_02x03_Odd_Even, J10 WAVESHAPE_CV, J11 5V_PATCH, J12 0V_PATCH, J13 RNG_CV, J14 RUNGLER_OUT, J15 LFO_TRI, J16 LFO_SQR, J17 LFO_RESET, J18 LFO_CV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

Commit message: Add files via upload
Parts:
- added C11: 100n, Capacitor_SMD:C_0805_2012Metric_Pad1.18x1.45mm_HandSolder, symbol Device:C
- added D16: 1N5819WS, Diode_SMD:D_SOD-323_HandSoldering, symbol Diode:1N5819WS
- added J19: Conn_01x02_Pin, Connector_JST:JST_EH_B2B-EH-A_1x02_P2.50mm_Vertical, symbol Connector:Conn_01x02_Pin
- D1, D10, D11, D13, D14, D15, D5, D6, D7, D8, D9: footprint Diode_THT:D_DO-41_SOD81_P2.54mm_Vertical_AnodeUp -> Diode_SMD:D_MiniMELF_Handsoldering
- D2, D3, D4: footprint Diode_SMD:D_SOD-323 -> Diode_SMD:D_SOD-323_HandSoldering
Connections:
- net +5V: now also C11.1, D16.1 (K)
- net GND: now also C11.2, J19.2 (Pin_2)
- new net: D16.2 (A), J19.1 (Pin_1)
Other:
- note added: "USB/External 5V"
